Commit message: urdf changes

File: thesis_description/urdf/gazebo.xacro (robot description, xacro)
@@ -1,4 +1,7 @@
 <?xml version="1.0" ?>
 <robot name="Thesis" xmlns:xacro="http://www.ros.org/wiki/xacro">
+  <gazebo reference="base_link">
+    <material>Gazebo/OrangeTransparent</material>
+  </gazebo>
   <gazebo reference="ruedatraseraizquierda">
     <mu1>0.5</mu1>
@@ -59,7 +62,7 @@
       <covariance_y>0.0001</covariance_y>
       <covariance_yaw>0.01</covariance_yaw>
-      <wheelSeparation>0.60</wheelSeparation>
-      <wheelDiameter>0.23</wheelDiameter>
-      <torque>40</torque>
+      <wheelSeparation>0.60</wheelSeparation> <!--Por corregir-->
+      <wheelDiameter>0.32766</wheelDiameter> <!--CORREGIDO-->
+      <torque>40</torque> <!--Por corregir-->
       <commandTopic>cmd_vel</commandTopic>
       <odometryTopic>odom</odometryTopic>

File: thesis_description/urdf/thesis.xacro (robot description, xacro)
@@ -14,14 +14,17 @@
     <color rgba="0 0 1 1"/>
   </material>
+  <material name="orange">
+    <color rgba="0.949 0.361 0.098 1"/>
+  </material>
   <!-- BGN - Robot description -->
   <m_link_mesh name="base_link"
               origin_rpy="1.5807 0 1.5807" origin_xyz="0 0 0.03"
-              mass="5.0"
-              ixx="1.3235" ixy="0" ixz="0"
-              iyy="1.3235" iyz="0"
-              izz="0.9655"
-              material="white"
+              mass="26.28"
+              ixx="0.8837" ixy="0" ixz="0"
+              iyy="2.6409" iyz="0"
+              izz="3.0534"
+              material="orange"
               meshfile="package://thesis_description/meshes/base.stl"
-              meshscale="0.001 0.001 0.001" />
+              meshscale="0.01 0.01 0.01" /> <!--SOLO FALTA ORIGIN_XYZ-->
   <joint name="cuerpo__ruedafrentederecha" type="continuous">
       <parent link="base_link"/>
@@ -31,6 +34,6 @@
   </joint>
   <m_link_mesh name="ruedafrentederecha"
-              origin_rpy="1.5807 0 3.1416" origin_xyz="0 0 0"
-              mass="2"
+              origin_rpy="1.5708 0 4.7124" origin_xyz="0 0 0"
+              mass="13.43"
               ixx="0.132" ixy="0" ixz="0"
               iyy="0.132" iyz="0"
@@ -38,5 +41,5 @@
               material="black"
               meshfile="package://thesis_description/meshes/Rueda.stl"
-              meshscale="0.0009 0.0009 0.0009" />
+              meshscale="0.01 0.01 0.01" /> <!--CORREGIDO-->
   <joint name="cuerpo__ruedatraseraderecha" type="continuous">
       <parent link="base_link"/>
@@ -46,6 +49,6 @@
   </joint>
   <m_link_mesh name="ruedatraseraderecha"
-              origin_rpy="1.5807 0 3.1416" origin_xyz="0 0 0"
-              mass="2"
+              origin_rpy="1.5708 0 4.7124" origin_xyz="0 0 0"
+              mass="13.43"
               ixx="0.132" ixy="0" ixz="0"
               iyy="0.132" iyz="0"
@@ -53,5 +56,5 @@
               material="black"
               meshfile="package://thesis_description/meshes/Rueda.stl"
-              meshscale="0.0009 0.0009 0.0009" />
+              meshscale="0.01 0.01 0.01" /> <!--CORREGIDO-->
   <joint name="cuerpo__ruedafrenteizquierda" type="continuous">
       <parent link="base_link"/>
@@ -61,6 +64,6 @@
   </joint>
   <m_link_mesh name="ruedafrenteizquierda"
-              origin_rpy="1.5807 0 3.1416" origin_xyz="0 0 0"
-              mass="2"
+              origin_rpy="1.5708 0 1.5708" origin_xyz="0 0 0"
+              mass="13.43"
               ixx="0.132" ixy="0" ixz="0"
               iyy="0.132" iyz="0"
@@ -68,5 +71,5 @@
               material="black"
               meshfile="package://thesis_description/meshes/Rueda.stl"
-              meshscale="0.0009 0.0009 0.0009" />
+              meshscale="0.01 0.01 0.01" /> <!--CORREGIDO-->
   <joint name="cuerpo__ruedatraseraizquierda" type="continuous">
       <parent link="base_link"/>
@@ -76,6 +79,6 @@
   </joint>
   <m_link_mesh name="ruedatraseraizquierda"
-              origin_rpy="1.5807 0 3.1416" origin_xyz="0 0 0"
-              mass="2"
+              origin_rpy="1.5708 0 1.5708" origin_xyz="0 0 0"
+              mass="13.43"
               ixx="0.132" ixy="0" ixz="0"
               iyy="0.132" iyz="0"
@@ -83,4 +86,4 @@
               material="black"
               meshfile="package://thesis_description/meshes/Rueda.stl"
-              meshscale="0.0009 0.0009 0.0009" />
+              meshscale="0.01 0.01 0.01" /> <!--CORREGIDO-->
 </robot>

Commit message: results included

File: thesis_description/urdf/gazebo.xacro (robot description, xacro)
@@ -2,9 +2,9 @@
 <robot name="Thesis" xmlns:xacro="http://www.ros.org/wiki/xacro">
   <gazebo reference="base_link">
-    <material>Gazebo/OrangeTransparent</material>
+    <material>Gazebo/Orange</material>
   </gazebo>
   <gazebo reference="ruedatraseraizquierda">
-    <mu1>0.5</mu1>
-    <mu2>0.5</mu2>
+    <mu1>0.9</mu1>
+    <mu2>0.9</mu2>
     <kp>500000.0</kp>
     <kd>10.0</kd>
@@ -15,6 +15,6 @@
   </gazebo>
   <gazebo reference="ruedafrentederecha">
-    <mu1>0.5</mu1>
-    <mu2>0.5</mu2>
+    <mu1>0.9</mu1>
+    <mu2>0.9</mu2>
     <kp>500000.0</kp>
     <kd>10.0</kd>
@@ -25,6 +25,6 @@
   </gazebo>
   <gazebo reference="ruedafrenteizquierda">
-    <mu1>0.5</mu1>
-    <mu2>0.5</mu2>
+    <mu1>0.9</mu1>
+    <mu2>0.9</mu2>
     <kp>500000.0</kp>
     <kd>10.0</kd>
@@ -35,7 +35,7 @@
   </gazebo>
   <gazebo reference="ruedatraseraderecha">
-    <mu1>0.5</mu1>
-    <mu2>0.5</mu2>
-    <kp>500000.0</kp>
+    <mu1>0.9</mu1>
+    <mu2>0.9</mu2>
+    <kp>1000000.0</kp>
     <kd>10.0</kd>
     <minDepth>0.001</minDepth>
@@ -62,7 +62,7 @@
       <covariance_y>0.0001</covariance_y>
       <covariance_yaw>0.01</covariance_yaw>
-      <wheelSeparation>0.60</wheelSeparation> <!--Por corregir-->
-      <wheelDiameter>0.32766</wheelDiameter> <!--CORREGIDO-->
-      <torque>40</torque> <!--Por corregir-->
+      <wheelSeparation>0.6910</wheelSeparation>
+      <wheelDiameter>0.32766</wheelDiameter>
+      <torque>100</torque>
       <commandTopic>cmd_vel</commandTopic>
       <odometryTopic>odom</odometryTopic>
@@ -71,3 +71,150 @@
     </plugin>
   </gazebo>
+  <!-- Hokuyo LiDAR -->
+  <gazebo reference="hokuyo_link">
+    <material>Gazebo/Blue</material>
+    <sensor type="ray" name="hokuyo_sensor">
+      <pose>0 0 0 1.5708 0 1.5708</pose>
+      <visualize>true</visualize>
+      <update_rate>40</update_rate>
+      <ray>
+        <scan>
+          <horizontal>
+            <samples>1080</samples>
+            <resolution>0.25</resolution>
+            <min_angle>-2.3562</min_angle>
+            <max_angle>2.3562</max_angle>
+          </horizontal>
+        </scan>
+        <range>
+          <min>0.10</min>
+          <max>30.0</max>
+          <resolution>0.001</resolution>
+        </range>
+        <noise>
+          <type>gaussian</type>
+          <mean>0.0</mean>
+          <stddev>0.01</stddev>
+        </noise>
+      </ray>
+      <plugin name="gazebo_ros_head_hokuyo_controller" filename="libgazebo_ros_laser.so">
+        <topicName>/laser_scan</topicName>
+        <frameName>hokuyo_link</frameName>
+      </plugin>
+    </sensor>
+  </gazebo>
+  <!-- Depth camera
+  <gazebo reference="depth_link">
+    <material>Gazebo/Grey</material>
+    <sensor name="depth_camera" type="depth">
+      <always_on>true</always_on>
+      <update_rate>15.0</update_rate>
+      <visualize>true</visualize>
+      <camera>
+        <horizontal_fov>1.919867</horizontal_fov>
+        <image>
+          <width>1280</width>
+          <height>720</height>
+          <format>R8G8B8</format>
+        </image>
+        <clip>
+          <near>0.02</near>
+          <far>300</far>
+        </clip>
+        <noise>
+          <type>gaussian</type>
+          <mean>0.0</mean>
+          <stddev>0.007</stddev>
+        </noise>
+      </camera>
+      <plugin name="depth_link_controller" filename="libgazebo_ros_openni_kinect.so">
+        <baseline>0.2</baseline>
+        <alwaysOn>true</alwaysOn>
+        <updateRate>1.0</updateRate>
+        <cameraName>depth_camera_ir</cameraName>
+        <imageTopicName>depth_camera/color/image_raw</imageTopicName>
+        <cameraInfoTopicName>/depth_camera/color/camera_info</cameraInfoTopicName>
+        <depthImageTopicName>/depth_camera/depth/image_raw</depthImageTopicName>
+        <depthImageInfoTopicName>/depth_camera/depth/camera_info</depthImageInfoTopicName>
+        <pointCloudTopicName>/depth_camera/depth/points</pointCloudTopicName>
+        <frameName>depth_link</frameName>
+        <pointCloudCutoff>0.3</pointCloudCutoff>
+        <pointCloudCutoffMax>20.0</pointCloudCutoffMax>
+        <distortionK1>0.00000001</distortionK1>
+        <distortionK2>0.00000001</distortionK2>
+        <distortionK3>0.00000001</distortionK3>
+        <distortionT1>0.00000001</distortionT1>
+        <distortionT2>0.00000001</distortionT2>
+        <CxPrime>658.8206787109375</CxPrime>
+        <Cx>658.8206787109375</Cx>
+        <Cy>372.25787353515625</Cy>
+        <focalLength>0</focalLength>
+        <hackBaseline>0</hackBaseline>
+      </plugin>
+    </sensor>
+  </gazebo>-->
+<!-- -->
+  <gazebo reference="depth_link">
+    <material>Gazebo/Grey</material>
+    <sensor name="depth_camera" type="depth">
+      <update_rate>15</update_rate>
+      <camera>
+        <horizontal_fov>1.919862</horizontal_fov>
+        <image>
+          <width>2560</width>
+          <height>720</height>
+          <format>R8G8B8</format>
+        </image>
+        <clip>
+          <near>0.05</near>
+          <far>3</far>
+        </clip>
+      </camera>
+      <plugin name="depth_link_controller" filename="libgazebo_ros_openni_kinect.so">
+        <baseline>0.2</baseline>
+        <alwaysOn>true</alwaysOn>
+        <updateRate>1.0</updateRate>
+        <cameraName>depth_camera_ir</cameraName>
+        <imageTopicName>depth_camera/color/image_raw</imageTopicName>
+        <cameraInfoTopicName>/depth_camera/color/camera_info</cameraInfoTopicName>
+        <depthImageTopicName>/depth_camera/depth/image_raw</depthImageTopicName>
+        <depthImageInfoTopicName>/depth_camera/depth/camera_info</depthImageInfoTopicName>
+        <pointCloudTopicName>/depth_camera/depth/points</pointCloudTopicName>
+        <frameName>depth_link</frameName>
+        <pointCloudCutoff>0.2</pointCloudCutoff>
+        <pointCloudCutoffMax>20.0</pointCloudCutoffMax>
+        <distortionK1>0.00000001</distortionK1>
+        <distortionK2>0.00000001</distortionK2>
+        <distortionK3>0.00000001</distortionK3>
+        <distortionT1>0.00000001</distortionT1>
+        <distortionT2>0.00000001</distortionT2>
+        <CxPrime>0</CxPrime>
+        <Cx>0</Cx>
+        <Cy>0</Cy>
+        <focalLength>0</focalLength>
+        <hackBaseline>0</hackBaseline>
+      </plugin>
+    </sensor>
+  </gazebo>
+  <!--IMU -->
+  <gazebo reference="imu_link">
+    <gravity>true</gravity>
+    <sensor name="imu_sensor" type="imu">
+      <always_on>true</always_on>
+      <update_rate>100</update_rate>
+      <visualize>true</visualize>
+      <topic>__default_topic__</topic>
+      <plugin filename="libgazebo_ros_imu_sensor.so" name="imu_plugin">
+        <topicName>imu</topicName>
+        <bodyName>imu_link</bodyName>
+        <updateRateHZ>10.0</updateRateHZ>
+        <gaussianNoise>0.0</gaussianNoise>
+        <xyzOffset>0 0 0</xyzOffset>
+        <rpyOffset>0 0 0</rpyOffset>
+        <frameName>imu_link</frameName>
+        <initialOrientationAsReference>false</initialOrientationAsReference>
+      </plugin>
+      <pose>0 0 0 0 0 0</pose>
+    </sensor>
+  </gazebo>
 </robot>

File: thesis_description/urdf/thesis.xacro (robot description, xacro)
@@ -14,4 +14,7 @@
     <color rgba="0 0 1 1"/>
   </material>
+  <material name="grey">
+    <color rgba="0.332 0.332 0.332 1"/>
+  </material>
   <material name="orange">
     <color rgba="0.949 0.361 0.098 1"/>
@@ -19,5 +22,5 @@
   <!-- BGN - Robot description -->
   <m_link_mesh name="base_link"
-              origin_rpy="1.5807 0 1.5807" origin_xyz="0 0 0.03"
+              origin_rpy="1.5807 0 1.5807" origin_xyz="0 0 0.2355"
               mass="26.28"
               ixx="0.8837" ixy="0" ixz="0"
@@ -26,9 +29,9 @@
               material="orange"
               meshfile="package://thesis_description/meshes/base.stl"
-              meshscale="0.01 0.01 0.01" /> <!--SOLO FALTA ORIGIN_XYZ-->
+              meshscale="0.010335 0.010335 0.010335" />
   <joint name="cuerpo__ruedafrentederecha" type="continuous">
       <parent link="base_link"/>
       <child link="ruedafrentederecha"/>
-      <origin xyz="0.21 -0.30 -0.05" rpy="0.0 0.0 0"/>
+      <origin xyz="0.311 -0.3455 0.1638" rpy="0.0 0.0 0"/>
       <axis xyz="0 1 0"/>
   </joint>
@@ -36,14 +39,14 @@
               origin_rpy="1.5708 0 4.7124" origin_xyz="0 0 0"
               mass="13.43"
-              ixx="0.132" ixy="0" ixz="0"
-              iyy="0.132" iyz="0"
-              izz="0.097"
+              ixx="0.1798" ixy="0" ixz="0"
+              iyy="0.1081" iyz="0"
+              izz="0.1798"
               material="black"
               meshfile="package://thesis_description/meshes/Rueda.stl"
-              meshscale="0.01 0.01 0.01" /> <!--CORREGIDO-->
+              meshscale="0.010335 0.010335 0.010335" />
   <joint name="cuerpo__ruedatraseraderecha" type="continuous">
       <parent link="base_link"/>
       <child link="ruedatraseraderecha"/>
-      <origin xyz="-0.20 -0.30 -0.05" rpy="0.0 0.0 0"/>
+      <origin xyz="-0.311 -0.3455 0.1638" rpy="0.0 0.0 0"/>
       <axis xyz="0 1 0"/>
   </joint>
@@ -51,14 +54,14 @@
               origin_rpy="1.5708 0 4.7124" origin_xyz="0 0 0"
               mass="13.43"
-              ixx="0.132" ixy="0" ixz="0"
-              iyy="0.132" iyz="0"
-              izz="0.097"
+              ixx="0.1798" ixy="0" ixz="0"
+              iyy="0.1081" iyz="0"
+              izz="0.1798"
               material="black"
               meshfile="package://thesis_description/meshes/Rueda.stl"
-              meshscale="0.01 0.01 0.01" /> <!--CORREGIDO-->
+              meshscale="0.010335 0.010335 0.010335" />
   <joint name="cuerpo__ruedafrenteizquierda" type="continuous">
       <parent link="base_link"/>
       <child link="ruedafrenteizquierda"/>
-      <origin xyz="0.21 0.30 -0.05" rpy="0.0 0.0 0"/>
+      <origin xyz="0.311 0.3455 0.1638" rpy="0.0 0.0 0"/>
       <axis xyz="0 1 0"/>
   </joint>
@@ -66,14 +69,14 @@
               origin_rpy="1.5708 0 1.5708" origin_xyz="0 0 0"
               mass="13.43"
-              ixx="0.132" ixy="0" ixz="0"
-              iyy="0.132" iyz="0"
-              izz="0.097"
+              ixx="0.1798" ixy="0" ixz="0"
+              iyy="0.1081" iyz="0"
+              izz="0.1798"
               material="black"
               meshfile="package://thesis_description/meshes/Rueda.stl"
-              meshscale="0.01 0.01 0.01" /> <!--CORREGIDO-->
+              meshscale="0.010335 0.010335 0.010335" />
   <joint name="cuerpo__ruedatraseraizquierda" type="continuous">
       <parent link="base_link"/>
       <child link="ruedatraseraizquierda"/>
-      <origin xyz="-0.20 0.30 -0.05" rpy="0.0 0.0 0"/>
+      <origin xyz="-0.311 0.3455 0.1638" rpy="0.0 0.0 0"/>
       <axis xyz="0 1 0"/>
   </joint>
@@ -81,9 +84,90 @@
               origin_rpy="1.5708 0 1.5708" origin_xyz="0 0 0"
               mass="13.43"
-              ixx="0.132" ixy="0" ixz="0"
-              iyy="0.132" iyz="0"
-              izz="0.097"
+              ixx="0.1798" ixy="0" ixz="0"
+              iyy="0.1081" iyz="0"
+              izz="0.1798"
               material="black"
               meshfile="package://thesis_description/meshes/Rueda.stl"
-              meshscale="0.01 0.01 0.01" /> <!--CORREGIDO-->
+              meshscale="0.010335 0.010335 0.010335" />
+  <!-- Hokuyo LiDAR -->
+  <joint name="hokuyo_joint" type="fixed">
+    <axis xyz="0 1 0" />
+    <origin xyz="0.4090 0 0.4430" rpy="0 0 0"/>
+    <parent link="base_link"/>
+    <child link="hokuyo_link"/>
+  </joint>
+  <link name="hokuyo_link">
+    <collision>
+      <origin xyz="0 0 0" rpy="1.5708 0 1.5708"/>
+      <geometry>
+        <mesh filename="package://thesis_description/meshes/LiDAR_2D.stl" scale="0.010335 0.010335 0.010335"/>
+      </geometry>
+    </collision>
+    <visual>
+      <origin xyz="0 0 0" rpy="1.5708 0 1.5708"/>
+      <geometry>
+        <mesh filename="package://thesis_description/meshes/LiDAR_2D.stl" scale="0.010335 0.010335 0.010335"/>
+      </geometry>
+      <material name="blue"/>
+    </visual>
+    <inertial>
+      <mass value="0.370" />
+      <origin xyz="0 0 0" rpy="1.5708 0 1.5708"/>
+      <inertia ixx="1e-6" ixy="0" ixz="0" iyy="1e-6" iyz="0" izz="1e-6" />
+    </inertial>z siguiente es 0.371
+  </link>
+  <!-- Depth camera -->
+  <joint name="depth_joint" type="fixed">
+    <axis xyz="0 1 0" />
+    <origin xyz="0.5 0 0.371" rpy="0 0 0"/>
+    <parent link="base_link"/>
+    <child link="depth_link"/>
+  </joint>
+  <link name="depth_link">
+    <collision>
+      <origin xyz="0 0 0" rpy="-0.0326 0 -1.5708"/>
+      <geometry>
+        <mesh filename="package://thesis_description/meshes/Camara_estereo.stl" scale="0.010335 0.010335 0.010335"/>
+      </geometry>
+    </collision>
+    <visual>
+      <origin xyz="0 0 0" rpy="-0.0326 0 -1.5708"/>
+      <geometry>
+        <mesh filename="package://thesis_description/meshes/Camara_estereo.stl" scale="0.010335 0.010335 0.010335"/>
+      </geometry>
+      <material name="grey"/>
+    </visual>
+    <inertial>
+      <mass value="1e-5" />
+      <origin xyz="0 0 0" rpy="-0.0326 0 -1.5708"/>
+      <inertia ixx="1e-6" ixy="0" ixz="0" iyy="1e-6" iyz="0" izz="1e-6" />
+    </inertial>
+  </link>
+  <!-- IMU -->
+  <joint name="imu_joint" type="fixed">
+    <axis xyz="0 1 0" />
+    <origin xyz="0 0 0" rpy="0 0 0"/>
+    <parent link="base_link"/>
+    <child link="imu_link"/>
+  </joint>
+  <link name="imu_link">
+    <collision>
+      <origin xyz="0 0 0" rpy="0 0 0"/>
+      <geometry>
+        <mesh filename="package://thesis_description/meshes/IMU.stl" scale="0.010335 0.010335 0.010335"/>
+      </geometry>
+    </collision>
+    <visual>
+      <origin xyz="0 0 0" rpy="0 0 0"/>
+      <geometry>
+        <mesh filename="package://thesis_description/meshes/IMU.stl" scale="0.010335 0.010335 0.010335"/>
+      </geometry>
+      <material name="grey"/>
+    </visual>
+    <inertial>
+      <mass value="1e-5" />
+      <origin xyz="0 0 0" rpy="0 0 0"/>
+      <inertia ixx="1e-6" ixy="0" ixz="0" iyy="1e-6" iyz="0" izz="1e-6" />
+    </inertial>
+  </link>
 </robot>

Commit message: results included

File: thesis_description/urdf/gazebo.xacro (robot description, xacro)
@@ -181,5 +181,5 @@
         <depthImageInfoTopicName>/depth_camera/depth/camera_info</depthImageInfoTopicName>
         <pointCloudTopicName>/depth_camera/depth/points</pointCloudTopicName>
-        <frameName>depth_link</frameName>
+        <frameName>depth_optical_link</frameName>
         <pointCloudCutoff>0.2</pointCloudCutoff>
         <pointCloudCutoffMax>20.0</pointCloudCutoffMax>

File: thesis_description/urdf/thesis.xacro (robot description, xacro)
@@ -144,4 +144,10 @@
     </inertial>
   </link>
+  <joint name="depth_optical_joint" type="fixed">
+    <origin xyz="0 0 0" rpy="-1.57 0 -1.57"/>
+    <parent link="depth_link"/>
+    <child link="depth_optical_link"/>
+  </joint>
+  <link name="depth_optical_link"/>
   <!-- IMU -->
   <joint name="imu_joint" type="fixed">
